File: VMU_HW_NEW_FILES/MCU.kicad_sch (KiCad schematic)
At the start: 24 parts, among them J6 ARM_JTAG_SWD_10, U2 SN65HVD233, U7 STM32F091RCTx

Commit message: MCU agian
Parts:
- removed C15, C16, C17, C18, C19, C3: 100n, Capacitor_SMD:C_0603_1608Metric, symbol Device:C
- removed C20, C21: 4.7u, Capacitor_SMD:C_0603_1608Metric, symbol Device:C
- removed C22: 10n, Capacitor_SMD:C_0603_1608Metric, symbol Device:C
- removed C23: 1u, Capacitor_SMD:C_0603_1608Metric, symbol Device:C
- removed D29: D_Schottky_x2_Serial_AKC, Package_TO_SOT_SMD:SOT-23, symbol KTHFS:D_Schottky_x2_Serial_AKC
- removed D30: GREEN, LED_SMD:LED_0603_1608Metric, symbol Device:LED
- removed D31: YELLOW, LED_SMD:LED_0603_1608Metric, symbol Device:LED
- removed D32: BLUE, LED_SMD:LED_0603_1608Metric, symbol Device:LED
- removed J6: ARM_JTAG_SWD_10, KTHFS:Atmel_ICP_connector, symbol KTHFS:ARM_JTAG_SWD_10
- removed R38, R39, R40: 1k, Resistor_SMD:R_0603_1608Metric, symbol Device:R
- removed R9: 120, Resistor_SMD:R_0603_1608Metric, symbol Device:R
- removed R?: 200, Resistor_SMD:R_0603_1608Metric, symbol Device:R
- removed R?: 51, Resistor_SMD:R_0603_1608Metric, symbol Device:R
- removed R?: 510, Resistor_SMD:R_0603_1608Metric, symbol Device:R
- removed U2: SN65HVD233, Package_SO:SOIC-8_3.9x4.9mm_P1.27mm, symbol Interface_CAN_LIN:SN65HVD233
- removed U7: STM32F091RCTx, Package_QFP:LQFP-64_10x10mm_P0.5mm, symbol MCU_ST_STM32F0:STM32F091RCTx
- added C?: 100n, symbol Device:C
- added C? (x5): 100n, Capacitor_SMD:C_0603_1608Metric, symbol Device:C
- added C?: 10n, Capacitor_SMD:C_0603_1608Metric, symbol Device:C
- added C? (x2): 4.7u, Capacitor_SMD:C_0805_2012Metric, symbol Device:C
- added C?: 1u, Capacitor_SMD:C_0805_2012Metric, symbol Device:C
- added J?: ARM_JTAG_SWD_10, symbol KTHFS:ARM_JTAG_SWD_10
- added U?: STM32F091RCTx, Package_QFP:LQFP-64_10x10mm_P0.5mm, symbol blocks-rescue:STM32F091RCTx-MCU_ST_STM32F0
- added U?: SN65HVD233, Package_SO:SOIC-8_3.9x4.9mm_P1.27mm, symbol Interface_CAN_LIN:SN65HVD233
Connections:
- net ANALOG_1: now also U?.15 (PA1)
- net ANALOG_10: now also U?.43 (PA10)
- net ANALOG_11: now also U?.44 (PA11)
- net ANALOG_12: now also U?.45 (PA12)
- net ANALOG_2: now also U?.16 (PA2)
- net ANALOG_3: now also U?.17 (PA3)
- net ANALOG_4: now also U?.20 (PA4)
- net ANALOG_5: now also U?.21 (PA5)
- net ANALOG_6: now also U?.22 (PA6)
- net ANALOG_7: now also U?.23 (PA7)
- net ANALOG_8: now also U?.41 (PA8)
- net ANALOG_9: now also U?.42 (PA9)
- net CAN1_H: now also U?.7 (CANH)
- net CAN1_L: now also U?.6 (CANL)
- net GND: now also C?.1, C?.2, C?.2, C?.2, C?.2, C?.2, C?.2, C?.2, C?.2, C?.2, J?.3 (GND), J?.5 (GND), J?.9 (GNDDetect), U?.12 (VSSA), U?.18 (VSS), U?.2 (GND), U?.31 (VSS), U?.47 (VSS), U?.5 (LBK), U?.63 (VSS), U?.8 (Rs)
- new net +3V3: C?.1, C?.1, C?.1, C?.1, C?.1, C?.1, C?.1, C?.1, C?.2, J?.1 (VTref), U?.13 (VDDA), U?.19 (VDD), U?.3 (VCC), U?.32 (VDD), U?.48 (VDDIO2), U?.64 (VDD)
- new net RX: U?.4 (R), U?.61 (PB8)
- new net TX: U?.1 (D), U?.62 (PB9)
- new net swdclk: J?.4 (SWDCLK/TCK), U?.49 (PA14)
- new net swdio: J?.2 (SWDIO/TMS), U?.46 (PA13)
- new net ~{reset}: C?.1, J?.10 (~{RESET}), U?.7 (NRST)
- no-connect marks 34 -> 3
Other:
- note added: "By shorting pin 5 and 8 to GND all SN65HVD23* transcievers will work"
- note added: "Decoupling capacitors"
- note added: "Layout notes:"
- note added: "VDD 100n caps should be placed close to each VDD pin. The 5.7u doesn't matter that much but it should be before the 3.3v trace splits to the VDD pins. VDDIO2 capacitros should be close to VDDIO2 pin VDDA capacitors should be close to VDDA pin"
- note removed: "CAN"
- note removed: "DNM"
- note removed: "Digital input 5 V Voltage divider used to scale down to aprox 3.3V"
- note removed: "MCU DECOUPLING"
- note removed: "MCU STATUS LEDS"
- note removed: "PIN 13"
- note removed: "PIN 19"
- note removed: "PIN 32"
- note removed: "PIN 48"
- note removed: "PIN 64"
- note removed: "SWD"
