File: VMU_HW_NEW_FILES/MCU.kicad_sch (KiCad schematic)
At the start: 24 parts, among them J6 ARM_JTAG_SWD_10, U2 SN65HVD233, U7 STM32F091RCTx

Commit message: MCU
New MCU
Parts:
- removed C15, C16, C17, C18, C19, C3: 100n, Capacitor_SMD:C_0603_1608Metric, symbol Device:C
- removed C20, C21: 4.7u, Capacitor_SMD:C_0603_1608Metric, symbol Device:C
- removed C22: 10n, Capacitor_SMD:C_0603_1608Metric, symbol Device:C
- removed C23: 1u, Capacitor_SMD:C_0603_1608Metric, symbol Device:C
- removed D29: D_Schottky_x2_Serial_AKC, Package_TO_SOT_SMD:SOT-23, symbol KTHFS:D_Schottky_x2_Serial_AKC
- removed D30: GREEN, LED_SMD:LED_0603_1608Metric, symbol Device:LED
- removed D31: YELLOW, LED_SMD:LED_0603_1608Metric, symbol Device:LED
- removed D32: BLUE, LED_SMD:LED_0603_1608Metric, symbol Device:LED
- removed J6: ARM_JTAG_SWD_10, KTHFS:Atmel_ICP_connector, symbol KTHFS:ARM_JTAG_SWD_10
- removed R38, R39, R40: 1k, Resistor_SMD:R_0603_1608Metric, symbol Device:R
- removed R9: 120, Resistor_SMD:R_0603_1608Metric, symbol Device:R
- removed R?: 200, Resistor_SMD:R_0603_1608Metric, symbol Device:R
- removed R?: 51, Resistor_SMD:R_0603_1608Metric, symbol Device:R
- removed R?: 510, Resistor_SMD:R_0603_1608Metric, symbol Device:R
- removed U2: SN65HVD233, Package_SO:SOIC-8_3.9x4.9mm_P1.27mm, symbol Interface_CAN_LIN:SN65HVD233
- removed U7: STM32F091RCTx, Package_QFP:LQFP-64_10x10mm_P0.5mm, symbol MCU_ST_STM32F0:STM32F091RCTx
- added C?: 100n, symbol Device:C
- added C? (x5): 100n, Capacitor_SMD:C_0603_1608Metric, symbol Device:C
- added C?: 10n, Capacitor_SMD:C_0603_1608Metric, symbol Device:C
- added C? (x2): 4.7u, Capacitor_SMD:C_0805_2012Metric, symbol Device:C
- added C?: 1u, Capacitor_SMD:C_0805_2012Metric, symbol Device:C
- added J?: ARM_JTAG_SWD_10, symbol KTHFS:ARM_JTAG_SWD_10
- added U?: STM32F091RCTx, Package_QFP:LQFP-64_10x10mm_P0.5mm, symbol blocks-rescue:STM32F091RCTx-MCU_ST_STM32F0
- added U?: SN65HVD233, Package_SO:SOIC-8_3.9x4.9mm_P1.27mm, symbol Interface_CAN_LIN:SN65HVD233
Connections:
- net ANALOG_1: now also U?.15 (PA1)
- net ANALOG_10: now also U?.43 (PA10)
- net ANALOG_11: now also U?.44 (PA11)
- net ANALOG_12: now also U?.45 (PA12)
- net ANALOG_2: now also U?.16 (PA2)
- net ANALOG_3: now also U?.17 (PA3)
- net ANALOG_4: now also U?.20 (PA4)
- net ANALOG_5: now also U?.21 (PA5)
- net ANALOG_6: now also U?.22 (PA6)
- net ANALOG_7: now also U?.23 (PA7)
- net ANALOG_8: now also U?.41 (PA8)
- net ANALOG_9: now also U?.42 (PA9)
- net CAN1_H: now also U?.7 (CANH)
- net CAN1_L: now also U?.6 (CANL)
- net GND: now also C?.1, C?.2, C?.2, C?.2, C?.2, C?.2, C?.2, C?.2, C?.2, C?.2, J?.3 (GND), J?.5 (GND), J?.9 (GNDDetect), U?.12 (VSSA), U?.18 (VSS), U?.2 (GND), U?.31 (VSS), U?.47 (VSS), U?.5 (LBK), U?.63 (VSS), U?.8 (Rs)
- new net +3V3: C?.1, C?.1, C?.1, C?.1, C?.1, C?.1, C?.1, C?.1, C?.2, J?.1 (VTref), U?.13 (VDDA), U?.19 (VDD), U?.3 (VCC), U?.32 (VDD), U?.48 (VDDIO2), U?.64 (VDD)
- new net RX: U?.4 (R), U?.61 (PB8)
- new net TX: U?.1 (D), U?.62 (PB9)
- new net swdclk: J?.4 (SWDCLK/TCK), U?.49 (PA14)
- new net swdio: J?.2 (SWDIO/TMS), U?.46 (PA13)
- new net ~{reset}: C?.1, J?.10 (~{RESET}), U?.7 (NRST)
- no-connect marks 34 -> 3
Other:
- note added: "By shorting pin 5 and 8 to GND all SN65HVD23* transcievers will work"
- note added: "Decoupling capacitors"
- note added: "Layout notes:"
- note added: "VDD 100n caps should be placed close to each VDD pin. The 5.7u doesn't matter that much but it should be before the 3.3v trace splits to the VDD pins. VDDIO2 capacitros should be close to VDDIO2 pin VDDA capacitors should be close to VDDA pin"
- note removed: "CAN"
- note removed: "DNM"
- note removed: "Digital input 5 V Voltage divider used to scale down to aprox 3.3V"
- note removed: "MCU DECOUPLING"
- note removed: "MCU STATUS LEDS"
- note removed: "PIN 13"
- note removed: "PIN 19"
- note removed: "PIN 32"
- note removed: "PIN 48"
- note removed: "PIN 64"
- note removed: "SWD"

Commit message: MCU
Snygga till MCU
Other:
- moved on the sheet: J?
Changed lines of the file:
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@@
   (junction (at 55.88 166.37) (diameter 0) (color 0 0 0 0)
   )
-  (junction (at 129.54 187.96) (diameter 0) (color 0 0 0 0)
+  (junction (at 44.577 125.095) (diameter 0) (color 0 0 0 0)
   )
   (junction (at 87.63 166.37) (diameter 0) (color 0 0 0 0)
@@
   (junction (at 151.384 39.116) (diameter 0) (color 0 0 0 0)
   )
-  (no_connect (at 144.78 173.99))
+  (no_connect (at 59.817 111.125))
   (no_connect (at 141.224 41.656))
-  (no_connect (at 144.78 176.53))
+  (no_connect (at 59.817 113.665))
   (wire (pts (xy 21.59 170.18) (xy 21.59 166.37))
     (stroke (width 0) (type default))
@@
     (stroke (width 0) (type default))
   )
-  (wire (pts (xy 144.78 163.83) (xy 156.21 163.83))
+  (wire (pts (xy 59.817 100.965) (xy 71.247 100.965))
     (stroke (width 0) (type default))
   )
@@
     (stroke (width 0) (type dash))
   )
-  (wire (pts (xy 129.54 189.23) (xy 129.54 187.96))
+  (wire (pts (xy 44.577 126.365) (xy 44.577 125.095))
     (stroke (width 0) (type default))
   )
@@
     (stroke (width 0) (type default))
   )
-  (wire (pts (xy 129.54 187.96) (xy 132.08 187.96))
+  (wire (pts (xy 44.577 125.095) (xy 47.117 125.095))
     (stroke (width 0) (type default))
   )
@@
     (stroke (width 0) (type default))
   )
-  (wire (pts (xy 132.08 156.21) (xy 132.08 154.94))
+  (wire (pts (xy 47.117 93.345) (xy 47.117 92.075))
     (stroke (width 0) (type default))
   )
@@
     (stroke (width 0) (type default))
   )
-  (wire (pts (xy 144.78 168.91) (xy 156.21 168.91))
+  (wire (pts (xy 59.817 106.045) (xy 71.247 106.045))
     (stroke (width 0) (type default))
   )
@@
     (stroke (width 0) (type dash))
   )
-  (wire (pts (xy 144.78 171.45) (xy 156.21 171.45))
+  (wire (pts (xy 59.817 108.585) (xy 71.247 108.585))
     (stroke (width 0) (type default))
   )
@@
     (stroke (width 0) (type default))
   )
-  (wire (pts (xy 129.54 187.96) (xy 129.54 186.69))
+  (wire (pts (xy 44.577 125.095) (xy 44.577 123.825))
     (stroke (width 0) (type default))
   )
@@
     (stroke (width 0) (type default))
   )
-  (wire (pts (xy 132.08 187.96) (xy 132.08 186.69))
+  (wire (pts (xy 47.117 125.095) (xy 47.117 123.825))
     (stroke (width 0) (type default))
   )
@@
     (stroke (width 0) (type default))
   )
+  (rectangle (start 19.05 87.884) (end 75.819 133.223)
+    (stroke (width 0) (type dash))
+    (fill (type none))
+  )
   (rectangle (start 242.316 119.38) (end 283.718 155.067)
     (stroke (width 0) (type dash))
@@
     (effects (font (size 1.27 1.27)) (justify right bottom))
   )
-  (label "swdclk" (at 156.21 168.91 180) (fields_autoplaced)
+  (label "swdclk" (at 71.247 106.045 180) (fields_autoplaced)
     (effects (font (size 1.27 1.27)) (justify right bottom))
   )
@@
     (effects (font (size 1.27 1.27)) (justify right bottom))
   )
-  (label "swdio" (at 156.21 171.45 180) (fields_autoplaced)
+  (label "swdio" (at 71.247 108.585 180) (fields_autoplaced)
     (effects (font (size 1.27 1.27)) (justify right bottom))
   )
-  (label "~{reset}" (at 156.21 163.83 180) (fields_autoplaced)
+  (label "~{reset}" (at 71.247 100.965 180) (fields_autoplaced)
     (effects (font (size 1.27 1.27)) (justify right bottom))
   )
@@
     )
   )
-  (symbol (lib_id "KTHFS:ARM_JTAG_SWD_10") (at 132.08 172.72 0) (unit 1)
+  (symbol (lib_id "KTHFS:ARM_JTAG_SWD_10") (at 47.117 109.855 0) (unit 1)
     (in_bom yes) (on_board yes) (dnp no)
-    (property "Reference" "J?" (at 120.8278 170.2816 0)
+    (property "Reference" "J?" (at 35.8648 107.4166 0)
       (effects (font (size 1.27 1.27)) (justify right))
     )
-    (property "Value" "ARM_JTAG_SWD_10" (at 125.73 156.21 0)
+    (property "Value" "ARM_JTAG_SWD_10" (at 40.767 93.345 0)
       (effects (font (size 1.27 1.27)) (justify right))
     )
-    (property "Footprint" "" (at 132.08 172.72 0)
+    (property "Footprint" "" (at 47.117 109.855 0)
       (effects (font (size 1.27 1.27)) hide)
     )
-    (property "Datasheet" "" (at 132.08 172.72 0)
+    (property "Datasheet" "" (at 47.117 109.855 0)
       (effects (font (size 1.27 1.27)) hide)
     )
@@
     )
   )
-  (symbol (lib_id "power:GND") (at 129.54 189.23 0) (unit 1)
+  (symbol (lib_id "power:GND") (at 44.577 126.365 0) (unit 1)
     (in_bom yes) (on_board yes) (dnp no)
-    (property "Reference" "#PWR?" (at 129.54 195.58 0)
+    (property "Reference" "#PWR?" (at 44.577 132.715 0)
       (effects (font (size 1.27 1.27)) hide)
     )
-    (property "Value" "GND" (at 129.667 193.6242 0)
+    (property "Value" "GND" (at 44.704 130.7592 0)
       (effects (font (size 1.27 1.27)))
     )
-    (property "Footprint" "" (at 129.54 189.23 0)
+    (property "Footprint" "" (at 44.577 126.365 0)
       (effects (font (size 1.27 1.27)) hide)
     )
-    (property "Datasheet" "" (at 129.54 189.23 0)
+    (property "Datasheet" "" (at 44.577 126.365 0)
       (effects (font (size 1.27 1.27)) hide)
     )
@@
     )
   )
-  (symbol (lib_id "blocks-rescue:+3.3V-power") (at 132.08 154.94 0) (unit 1)
+  (symbol (lib_id "blocks-rescue:+3.3V-power") (at 47.117 92.075 0) (unit 1)
     (in_bom yes) (on_board yes) (dnp no)
-    (property "Reference" "#PWR?" (at 132.08 158.75 0)
+    (property "Reference" "#PWR?" (at 47.117 95.885 0)
       (effects (font (size 1.27 1.27)) hide)
     )
-    (property "Value" "+3.3V" (at 132.461 150.5458 0)
+    (property "Value" "+3.3V" (at 47.498 87.6808 0)
       (effects (font (size 1.27 1.27)))
     )
-    (property "Footprint" "" (at 132.08 154.94 0)
+    (property "Footprint" "" (at 47.117 92.075 0)
       (effects (font (size 1.27 1.27)) hide)
     )
-    (property "Datasheet" "" (at 132.08 154.94 0)
+    (property "Datasheet" "" (at 47.117 92.075 0)
       (effects (font (size 1.27 1.27)) hide)
     )

Commit message: MCU FIX TORE
Parts:
- added R9: R, symbol Device:R
Connections:
- net +3V3: now also R9.1
- net ANALOG_1: now also U?.14 (PA0); no longer U?.15 (PA1)
- net ANALOG_10: now also U?.9 (PC1); no longer U?.43 (PA10)
- net ANALOG_11: now also U?.10 (PC2); no longer U?.44 (PA11)
- net ANALOG_12: now also U?.11 (PC3); no longer U?.45 (PA12)
- net ANALOG_2: now also U?.15 (PA1); no longer U?.16 (PA2)
- net ANALOG_3: now also U?.16 (PA2); no longer U?.17 (PA3)
- net ANALOG_4: now also U?.17 (PA3); no longer U?.20 (PA4)
- net ANALOG_5: now also U?.20 (PA4); no longer U?.21 (PA5)
- net ANALOG_6: now also U?.21 (PA5); no longer U?.22 (PA6)
- net ANALOG_7: now also U?.22 (PA6); no longer U?.23 (PA7)
- net ANALOG_8: now also U?.23 (PA7); no longer U?.41 (PA8)
- net ANALOG_9: now also U?.8 (PC0); no longer U?.42 (PA9)
