File: VMU_HW_NEW_FILES/SIGNAL_CONDITIONING_VMU.kicad_sch (KiCad schematic)
At the start: 78 parts, among them U2 TLV9064, U4 TLV9064, U6 TLV9064

Commit message: Update SIGNAL_CONDITIONING_VMU.kicad_sch
Parts:
- removed C? (x3): 100n, Capacitor_SMD:C_0603_1608Metric, symbol Device:C
- added C?: 100n, Capacitor_SMD:C_0603_1608Metric, symbol Device:C
- added C?: 10n, Capacitor_SMD:C_0603_1608Metric, symbol Device:C
- added C?: 4.7u, Capacitor_SMD:C_0805_2012Metric, symbol Device:C
Connections:
- net +3V3: now also U2.4 (V+), U4.4 (V+), U6.4 (V+), C?.1, C?.1, C?.1
- net GND: now also C?.2, C?.2, C?.2
Other:
- note added: "Decoupling capacitors"
- note removed: "hej"
