File: VMU/VMU.kicad_pcb (KiCad board)
At the start: 4 copper layers, 154.9 x 127 mm, 74 parts, among them J1 Conn_01x04_Pin, J10 Conn_01x03_Pin, J11 Conn_01x03_Pin, J12 Conn_01x04_Pin, J13 Conn_01x04_Pin, J14 Conn_01x06_Pin, J15 ARM_JTAG_SWD_10, J16 Conn_01x02_Pin, J2 Conn_01x03_Pin, J3 Conn_01x03_Pin, J4 Conn_01x03_Pin, J5 Conn_01x03_Pin, J6 Conn_01x03_Pin, J7 Conn_01x08_Pin, J8 Conn_01x08_Pin, J9 Conn_01x03_Pin, U1 TLV9064, U2 TLV9064, U3 ADP150AUJZ-3.3-R7, U4 SN65HVD233, U5 STM32F091RCTx, Y1 Crystal_GND24

Commit message: sdfsd
Parts:
- removed C10, C11, C12, C13, C8, C9: 10n, Capacitor_SMD:C_0603_1608Metric_Pad1.08x0.95mm_HandSolder
- removed J10, J11, J5, J6, J9: Conn_01x03_Pin, KTHFS:Wurth-WBT_2.54_male_angle_3
- removed J12, J13: Conn_01x04_Pin, KTHFS:Wurth-WTB_2.54_male_angle_4
- removed J14: Conn_01x06_Pin, KTHFS:Wurth-WBT_2.54_male_angle_6
- J1: value Conn_01x04_Pin -> TBL009-254-14GY-2GY; footprint KTHFS:Wurth-WTB_2.54_male_angle_4 -> KTHFS:TBL00925414GY2GY
- J2, J3, J4: value Conn_01x03_Pin -> TBL009-254-14GY-2GY; footprint KTHFS:Wurth-WBT_2.54_male_angle_3 -> KTHFS:TBL00925414GY2GY
- JP1, JP2, JP3, JP4: footprint Connector_PinHeader_2.54mm:PinHeader_1x03_P2.54mm_Vertical -> Jumper:SolderJumper-3_P2.0mm_Open_TrianglePad1.0x1.5mm_NumberLabels
- moved JP1 51.1 mm to (144.7, 91.5)
- moved J2 47.2 mm to (126.3, 78.2), turned to 180 degrees
- moved J1 33.1 mm to (165.5, 78.2)
- moved J3 27.6 mm to (133.1, 126.6)
- moved J4 25.3 mm to (95.0, 126.6)
- moved J15 11.9 mm to (164.6, 109.2), turned to 90 degrees
- moved C14 11.7 mm to (179.0, 125.6)
- moved C18 11.7 mm to (179.0, 135.6)
- moved R5 11.7 mm to (187.7, 125.6)
- moved R9 11.7 mm to (187.7, 135.6)
- moved C15 11.7 mm to (179.0, 128.1)
- moved C16 11.7 mm to (179.0, 130.6)
- moved C17 11.7 mm to (179.0, 133.1)
- moved C19 11.7 mm to (179.0, 138.2)
- moved R6 11.7 mm to (187.7, 128.1)
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Connections:
- F4 pad 2: /DIGITAL_SUPPLY_1 -> /DIGITAL_SUPPLY_3
- F5 pad 2: /SUPPLY_5 -> /SUPPLY_6
- J1 pad 1: /battery_in -> /SUPPLY_1
- J1 pad 2: /CAN1_H -> /SUPPLY_1
- J1 pad 3: /CAN1_L -> /ANALOG_1_SIGNAL
- J1 pad 4: GND -> /ANALOG_1_SIGNAL
- J16 pad 1: /DIGITAL_SUPPLY_1 -> /PB_SUPPLY
- J2 pad 1: /SUPPLY_1 -> /SUPPLY_5
- J2 pad 2: /ANALOG_1_SIGNAL -> /SUPPLY_5
- J2 pad 3: GND -> /ANALOG_5_SIGNAL
- J3 pad 1: /SUPPLY_2 -> /GPIO_SPLY_5
- J3 pad 2: /ANALOG_2_SIGNAL -> /GPIO_SPLY_5
- J3 pad 3: GND -> /GPIO_SPLY_6
- J4 pad 1: /SUPPLY_3 -> /battery_in
- J4 pad 2: /ANALOG_3_SIGNAL -> /battery_in
- J4 pad 3: GND -> /CAN1_H
- U5 pad 33: unconnected-(U5-PB12-Pad33) -> /GPIO_SPLY_1
- U5 pad 34: unconnected-(U5-PB13-Pad34) -> /GPIO_SPLY_2
- U5 pad 35: unconnected-(U5-PB14-Pad35) -> /GPIO_SPLY_3
- U5 pad 36: unconnected-(U5-PB15-Pad36) -> /GPIO_SPLY_4
- U5 pad 37: unconnected-(U5-PC6-Pad37) -> /GPIO_SPLY_5
- U5 pad 38: unconnected-(U5-PC7-Pad38) -> /GPIO_SPLY_6
- U5 pad 39: unconnected-(U5-PC8-Pad39) -> /GPIO_SPLY_7
- U5 pad 40: unconnected-(U5-PC9-Pad40) -> /GPIO_SPLY_8
Other:
- board size 154.9 x 127 mm -> 76.2 x 53.3 mm

Commit message: Adad
a
Parts:
- removed C16, C17: 36pF, Capacitor_SMD:C_0603_1608Metric_Pad1.08x0.95mm_HandSolder
- removed R9: 0, Resistor_SMD:R_0603_1608Metric_Pad0.98x0.95mm_HandSolder
- removed Y1: Crystal_GND24, Crystal:Crystal_SMD_3225-4Pin_3.2x2.5mm_HandSoldering
- moved JP4 106.7 mm to (99.2, 115.8)
- moved F2 105.3 mm to (105.7, 118.4), turned to 180 degrees
- moved U4 104.6 mm to (112.5, 90.2)
- moved F3 100.5 mm to (109.7, 118.4), turned to 180 degrees
- moved JP3 90.4 mm to (111.4, 115.8)
- moved J1 86.6 mm to (94.0, 127.0), turned to 0 degrees
- moved C24 86.4 mm to (120.5, 104.4), turned to 90 degrees
- moved J4 85.4 mm to (165.4, 78.2), turned to 180 degrees
- moved JP2 81.1 mm to (117.5, 115.8)
- moved C14 79.5 mm to (107.8, 90.3), turned to -90 degrees
- moved R2 78.6 mm to (117.4, 90.3), turned to -90 degrees
- moved F5 76.0 mm to (129.5, 88.1), turned to -90 degrees
- moved F4 72.9 mm to (132.5, 88.1), turned to -90 degrees
- moved C23 70.5 mm to (137.6, 91.9)
- moved C20 69.6 mm to (117.1, 104.4), turned to 90 degrees
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Other:
- outline, holes or cut-outs redrawn

Commit message: sadsadsa
Parts:
- moved D5 73.0 mm to (93.1, 95.7), turned to 90 degrees
- moved D6 71.3 mm to (94.7, 95.7), turned to 90 degrees
- moved R4 70.0 mm to (93.2, 99.2), turned to 90 degrees
- moved D7 69.3 mm to (96.5, 95.7), turned to 90 degrees
- moved R5 68.3 mm to (94.7, 99.2), turned to 90 degrees
- moved R6 66.2 mm to (96.5, 99.3), turned to 90 degrees
- moved JP4 39.7 mm to (138.9, 114.3), turned to 180 degrees
- moved C6 27.9 mm to (159.0, 113.8), turned to 90 degrees
- moved F2 27.6 mm to (132.5, 111.8), turned to 0 degrees
- moved JP1 27.5 mm to (132.8, 114.3), turned to 180 degrees
- moved C7 26.1 mm to (160.7, 113.8), turned to 90 degrees
- moved U3 25.6 mm to (164.1, 113.8), turned to 180 degrees
- moved J16 24.1 mm to (109.7, 110.5), turned to 180 degrees
- moved J15 23.9 mm to (94.8, 108.4), turned to -90 degrees
- moved C1 17.4 mm to (138.9, 107.4), turned to 180 degrees
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Connections:
- F5 pad 2: /SUPPLY_6 -> /SUPPLY_8
Routing:
- net +3.3V: track 0.00 -> 7.51 mm, vias 0 -> 1
- net /I2C_SDA: track 0.00 -> 5.08 mm
- net /I2C_SCL: track 0.00 -> 5.08 mm
- net /GPIO_SPLY_6: track 0.00 -> 5.08 mm
- net /GPIO_SPLY_5: track 0.00 -> 5.08 mm
- net /DIGITAL_SUPPLY_1: track 0.00 -> 5.08 mm
- net +5V: track 0.00 -> 2.36 mm
- added copper zone on In2.Cu, net +3.3V
- added copper zone on B.Cu, net GND
- added copper zone on F.Cu, net GND
- added copper zone on In1.Cu, net GND
Other:
- outline, holes or cut-outs redrawn

Commit message: RotingV1
Parts:
- moved JP3 6.77 mm to (111.2, 114.5)
- moved JP2 6.08 mm to (118.0, 114.4)
- moved C19 4.35 mm to (123.4, 92.0)
- moved C23 2.95 mm to (125.0, 90.2)
- moved C18 0.89 mm to (119.8, 92.0)
- moved F3 0.40 mm to (119.7, 111.5)
- moved J2 0.28 mm to (125.3, 81.6)
Routing:
- net +5V: track 2.36 -> 101.9 mm, vias 0 -> 2
- net /GPIO_SPLY_2: track 0.00 -> 95.4 mm, vias 0 -> 6
- net /CAN1_H: track 0.00 -> 73.6 mm
- net /CAN1_L: track 0.00 -> 71.2 mm
- net +24V: track 0.00 -> 68.1 mm, vias 0 -> 2
- net Net-(JP1-A): track 0.00 -> 67.9 mm, vias 0 -> 2
- net /GPIO_SPLY_4: track 0.00 -> 65.1 mm
- net /GPIO_SPLY_1: track 0.00 -> 61.2 mm, vias 0 -> 2
- net /SUPPLY_1: track 0.00 -> 60.1 mm
- net Net-(JP1-B): track 0.00 -> 56.1 mm, vias 0 -> 3
- net +3.3V: track 7.51 -> 63.0 mm, vias 1 -> 10
- net /GPIO_SPLY_3: track 0.00 -> 54.5 mm
- net /SUPPLY_8: track 0.00 -> 53.6 mm, vias 0 -> 2
- net /MCU/~{reset}: track 0.00 -> 48.4 mm, vias 0 -> 2
- net /MCU/STATUS_LED_3_LED: track 0.00 -> 47.2 mm, vias 0 -> 2
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
Commit message: RoutingV2
Parts:
- moved R4 73.1 mm to (165.6, 89.0), turned to 180 degrees
- moved R5 71.3 mm to (165.7, 92.5), turned to 180 degrees
- moved U3 70.9 mm to (93.2, 112.2), turned to 90 degrees
- moved R6 69.8 mm to (165.8, 90.8), turned to 180 degrees
- moved D5 69.3 mm to (162.1, 89.0), turned to 180 degrees
- moved C4 68.5 mm to (96.0, 112.5), turned to -90 degrees
- moved D6 67.6 mm to (162.3, 92.5), turned to 180 degrees
- moved C7 67.6 mm to (93.2, 109.2), turned to 0 degrees
- moved C5 66.9 mm to (97.8, 112.5), turned to -90 degrees
- moved C6 66.1 mm to (93.2, 107.5), turned to 0 degrees
- moved D7 65.9 mm to (162.2, 90.8), turned to 180 degrees
- moved R1 64.2 mm to (96.0, 108.8), turned to 90 degrees
- moved D4 62.6 mm to (97.8, 108.8), turned to 90 degrees
- moved D3 60.2 mm to (96.5, 105.2), turned to 180 degrees
- moved J1 53.1 mm to (125.5, 80.0), turned to 180 degrees
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Connections:
- F4 pad 2: /DIGITAL_SUPPLY_3 -> /DIGITAL_SUPPLY_1
- F5 pad 2: /SUPPLY_8 -> /PB_SUPPLY
- J1 pad 1: /SUPPLY_1 -> GND
- J1 pad 10: /ANALOG_2_SIGNAL -> /SUPPLY_4
- J1 pad 13: /SUPPLY_3 -> /ANALOG_3_SIGNAL
- J1 pad 14: /SUPPLY_3 -> /ANALOG_3_SIGNAL
- J1 pad 15: /ANALOG_3_SIGNAL -> /SUPPLY_3
- J1 pad 16: /ANALOG_3_SIGNAL -> /SUPPLY_3
- J1 pad 19: /SUPPLY_4 -> /ANALOG_2_SIGNAL
- J1 pad 2: /SUPPLY_1 -> GND
- J1 pad 20: /SUPPLY_4 -> /ANALOG_2_SIGNAL
- J1 pad 21: /ANALOG_4_SIGNAL -> /SUPPLY_2
- J1 pad 22: /ANALOG_4_SIGNAL -> /SUPPLY_2
- J1 pad 25: /GPIO_SPLY_2 -> /ANALOG_1_SIGNAL
- J1 pad 26: /GPIO_SPLY_2 -> /ANALOG_1_SIGNAL
- J1 pad 27: GND -> /SUPPLY_1
- J1 pad 28: GND -> /SUPPLY_1
- J1 pad 3: /ANALOG_1_SIGNAL -> /GPIO_SPLY_2
- J1 pad 4: /ANALOG_1_SIGNAL -> /GPIO_SPLY_2
- J1 pad 7: /SUPPLY_2 -> /ANALOG_4_SIGNAL
- J1 pad 8: /SUPPLY_2 -> /ANALOG_4_SIGNAL
- J1 pad 9: /ANALOG_2_SIGNAL -> /SUPPLY_4
- J2 pad 1: /SUPPLY_5 -> GND
- J2 pad 10: /ANALOG_6_SIGNAL -> /PB_SUPPLY
- J2 pad 13: /SUPPLY_7 -> /ANALOG_7_SIGNAL
- J2 pad 14: /SUPPLY_7 -> /ANALOG_7_SIGNAL
- J2 pad 15: /ANALOG_7_SIGNAL -> /PB_SUPPLY
- J2 pad 16: /ANALOG_7_SIGNAL -> /PB_SUPPLY
- J2 pad 19: /SUPPLY_8 -> /ANALOG_6_SIGNAL
- J2 pad 2: /SUPPLY_5 -> GND
- J2 pad 20: /SUPPLY_8 -> /ANALOG_6_SIGNAL
- J2 pad 21: /ANALOG_8_SIGNAL -> /PB_SUPPLY
- J2 pad 22: /ANALOG_8_SIGNAL -> /PB_SUPPLY
- J2 pad 25: /GPIO_SPLY_1 -> /ANALOG_5_SIGNAL
- J2 pad 26: /GPIO_SPLY_1 -> /ANALOG_5_SIGNAL
- J2 pad 27: GND -> /PB_SUPPLY
- J2 pad 28: GND -> /PB_SUPPLY
- J2 pad 3: /ANALOG_5_SIGNAL -> /GPIO_SPLY_1
- J2 pad 4: /ANALOG_5_SIGNAL -> /GPIO_SPLY_1
- J2 pad 7: /SUPPLY_6 -> /ANALOG_8_SIGNAL
- J2 pad 8: /SUPPLY_6 -> /ANALOG_8_SIGNAL
- J2 pad 9: /ANALOG_6_SIGNAL -> /PB_SUPPLY
- J3 pad 19: /DIGITAL_SUPPLY_2 -> /DIGITAL_SUPPLY_1
- J3 pad 20: /DIGITAL_SUPPLY_2 -> /DIGITAL_SUPPLY_1
- J4 pad 1: /battery_in -> GND
- J4 pad 10: /GPIO_SPLY_4 -> /SPI_SCLK
- J4 pad 11: /GPIO_SPLY_3 -> /SPI_MOSI
- J4 pad 12: /GPIO_SPLY_3 -> /SPI_MOSI
- J4 pad 13: /DIGITAL_SUPPLY_3 -> /SPI_MISO
- J4 pad 14: /DIGITAL_SUPPLY_3 -> /SPI_MISO
- J4 pad 15: /SPI_MISO -> /DIGITAL_SUPPLY_1
- J4 pad 16: /SPI_MISO -> /DIGITAL_SUPPLY_1
- J4 pad 17: /SPI_MOSI -> /GPIO_SPLY_3
- J4 pad 18: /SPI_MOSI -> /GPIO_SPLY_3
- J4 pad 19: /SPI_SCLK -> /GPIO_SPLY_4
- J4 pad 2: /battery_in -> GND
- J4 pad 20: /SPI_SCLK -> /GPIO_SPLY_4
- J4 pad 21: /SPI_~{CS} -> GND
- J4 pad 22: /SPI_~{CS} -> GND
- J4 pad 23: GND -> /CAN1_L
- J4 pad 24: GND -> /CAN1_L
- J4 pad 25: GND -> /CAN1_H
- J4 pad 26: GND -> /CAN1_H
- J4 pad 27: GND -> /battery_in
- J4 pad 28: GND -> /battery_in
- J4 pad 3: /CAN1_H -> GND
- J4 pad 4: /CAN1_H -> GND
- J4 pad 5: /CAN1_L -> GND
- J4 pad 6: /CAN1_L -> GND
- J4 pad 7: GND -> /SPI_~{CS}
- J4 pad 8: GND -> /SPI_~{CS}
- J4 pad 9: /GPIO_SPLY_4 -> /SPI_SCLK
- U5 pad 10: /MCU/ANALOG_3 -> /MCU/ANALOG_6
- U5 pad 11: /MCU/ANALOG_4 -> /MCU/ANALOG_5
- U5 pad 14: /MCU/ANALOG_5 -> /MCU/ANALOG_4
- U5 pad 15: /MCU/ANALOG_6 -> /MCU/ANALOG_3
- U5 pad 16: /MCU/ANALOG_7 -> /MCU/ANALOG_2
- U5 pad 17: /MCU/ANALOG_8 -> /MCU/ANALOG_1
- U5 pad 8: /MCU/ANALOG_1 -> /MCU/ANALOG_8
- U5 pad 9: /MCU/ANALOG_2 -> /MCU/ANALOG_7
Routing:
- net /GPIO_SPLY_2: track 95.4 -> 5.08 mm, vias 6 -> 0
- net /DIGITAL_SUPPLY_1: track 5.08 -> 88.4 mm, vias 0 -> 1
- net /I2C_SDA: track 7.36 -> 70.6 mm, vias 0 -> 2
- net /GPIO_SPLY_4: track 65.1 -> 5.08 mm
- net +5V: track 101.9 -> 43.0 mm, vias 2 -> 8
- net /I2C_SCL: track 7.47 -> 64.1 mm, vias 0 -> 2
- net /GPIO_SPLY_1: track 61.2 -> 5.08 mm, vias 2 -> 0
- net /SUPPLY_8: track 53.6 -> 0.00 mm, vias 2 -> 0
- net Net-(JP1-A): track 67.9 -> 17.6 mm
- net /GPIO_SPLY_3: track 54.5 -> 5.08 mm
- net /PB_SUPPLY: track 0.00 -> 48.0 mm
- net +24V: track 68.1 -> 109.6 mm, vias 2 -> 3
- net Net-(JP1-B): track 56.1 -> 19.0 mm, vias 3 -> 2
- net /MCU/ANALOG_8: track 1.27 -> 32.7 mm
- net /SUPPLY_1: track 60.1 -> 29.1 mm
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- added copper zone on In2.Cu, net +5V
Other:
- board size 76.2 x 53.3 mm -> 76.2 x 53.8 mm

Commit message: Update
Parts:
- moved R5 74.9 mm to (93.5, 112.4), turned to 90 degrees
- moved R6 73.8 mm to (95.2, 112.4), turned to 90 degrees
- moved R4 72.4 mm to (97.0, 112.4), turned to 90 degrees
- moved D6 70.9 mm to (93.2, 108.6), turned to 90 degrees
- moved D7 69.3 mm to (95.2, 108.6), turned to 90 degrees
- moved D5 67.8 mm to (97.2, 108.7), turned to 90 degrees
- moved C4 67.5 mm to (163.5, 114.0)
- moved C5 67.5 mm to (165.2, 114.0)
- moved D3 64.3 mm to (160.5, 111.0), turned to 0 degrees
- moved D4 62.5 mm to (160.0, 114.0)
- moved R1 62.5 mm to (158.2, 114.0)
- moved D1 23.6 mm to (163.0, 88.8), turned to 0 degrees
- moved F1 21.3 mm to (163.0, 91.0), turned to 180 degrees
- moved D2 19.4 mm to (163.0, 93.2), turned to 180 degrees
- moved C3 17.3 mm to (163.0, 95.2), turned to 180 degrees
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Routing:
- net /GPIO_SPLY_1: track 5.08 -> 71.1 mm, vias 0 -> 2
- net /GPIO_SPLY_4: track 5.08 -> 65.3 mm, vias 0 -> 2
- net GND: track 27.3 -> 84.1 mm, vias 7 -> 19
- net /GPIO_SPLY_3: track 5.08 -> 60.8 mm, vias 0 -> 2
- net /GPIO_SPLY_5: track 5.08 -> 49.8 mm, vias 0 -> 2
- net /GPIO_SPLY_6: track 5.08 -> 47.9 mm, vias 0 -> 2
- net /CAN1_L: track 47.3 -> 68.5 mm
- net /GPIO_SPLY_2: track 5.08 -> 24.3 mm, vias 0 -> 1
- net /battery_in: track 21.9 -> 36.8 mm, vias 0 -> 1
- net +24V: track 109.6 -> 99.1 mm, vias 3 -> 1
- net /MCU/STATUS_LED_1_LED: track 37.7 -> 45.9 mm
- net /CAN1_H: track 52.6 -> 60.1 mm, vias 0 -> 1
- net +3.3V: track 61.5 -> 55.0 mm, vias 5 -> 9
- net Net-(VR1-OUT): track 10.3 -> 4.70 mm
- net /DIGITAL_SUPPLY_1: track 88.4 -> 93.8 mm
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Other:
- board size 76.2 x 53.8 mm -> 76.2 x 53.3 mm

Commit message: fiixes
Changed lines of the file:
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@@
     (property "ki_keywords" "diode TVS thyrector")
     (attr smd)
-    (fp_text reference "D2" (at 3.2 0 90) (layer "F.SilkS")
+    (fp_text reference "D2" (at 3.2 0 180) (layer "F.SilkS")
         (effects (font (size 1 1) (thickness 0.15)))
     )
@@
     (property "ki_keywords" "fuse")
     (attr smd)
-    (fp_text reference "F1" (at 3 0.25 90) (layer "F.SilkS")
+    (fp_text reference "F1" (at 3.2 0 180) (layer "F.SilkS")
         (effects (font (size 1 1) (thickness 0.15)))
     )
@@
     (property "ki_keywords" "quad opamp")
     (attr smd)
-    (fp_text reference "U2" (at -0.25 5.5 90) (layer "F.SilkS")
+    (fp_text reference "U2" (at -2.85 5.4 180) (layer "F.SilkS")
         (effects (font (size 1 1) (thickness 0.15)))
     )
@@
     (property "ki_keywords" "cap capacitor")
     (attr smd)
-    (fp_text reference "C3" (at 3 0 90) (layer "F.SilkS")
+    (fp_text reference "C3" (at 3.2 -0.05 180) (layer "F.SilkS")
         (effects (font (size 1 1) (thickness 0.15)))
     )
@@
     (property "ki_keywords" "fuse")
     (attr smd)
-    (fp_text reference "F4" (at -1.25 -2 90) (layer "F.SilkS")
+    (fp_text reference "F4" (at -2.85 0.05 180) (layer "F.SilkS")
         (effects (font (size 1 1) (thickness 0.15)))
     )
@@
     (property "ki_keywords" "diode Schottky")
     (attr smd)
-    (fp_text reference "D1" (at -3.25 0 90) (layer "F.SilkS")
+    (fp_text reference "D1" (at -3.2 0.15 180) (layer "F.SilkS")
         (effects (font (size 1 1) (thickness 0.15)))
     )
@@
     (pts (xy 174.678974 74.8875) (xy 174.686554 128.22508))
     (height -9.732213)
-    (gr_text "53.3376 mm" (at 185.564977 101.554744 270.0081425) (layer "User.1")
+    (gr_text "53,3376 mm" (at 185.564977 101.554744 270.0081425) (layer "User.1")
       (effects (font (size 1 1) (thickness 0.15)))
     )
@@
     (pts (xy 167.64758 128.52158) (xy 91.44242 128.52158))
     (height -10.97842)
-    (gr_text "76.2052 mm" (at 129.545 138.35) (layer "User.1")
+    (gr_text "76,2052 mm" (at 129.545 138.35) (layer "User.1")
       (effects (font (size 1 1) (thickness 0.15)))
     )
@@
   (segment (start 143.93 80) (end 143.93 85.08) (width 0.5) (layer "B.Cu") (net 95))
   (zone (net 2) (net_name "GND") (layers "F.Cu" "In1.Cu" "B.Cu") (hatch edge 0.5)
-    (connect_pads (clearance 0.5))
-    (min_thickness 0.25) (filled_areas_thickness no)
+    (connect_pads (clearance 0.2))
+    (min_thickness 0.2) (filled_areas_thickness no)
     (fill yes (thermal_gap 0.5) (thermal_bridge_width 0.5))
     (polygon
@@
   (zone (net 1) (net_name "+5V") (layer "In2.Cu") (hatch edge 0.5)
     (priority 2)
-    (connect_pads (clearance 0.5))
-    (min_thickness 0.25) (filled_areas_thickness no)
+    (connect_pads (clearance 0.2))
+    (min_thickness 0.2) (filled_areas_thickness no)
     (fill yes (thermal_gap 0.5) (thermal_bridge_width 0.5))
     (polygon
@@
   (zone (net 4) (net_name "+3.3V") (layer "In2.Cu") (hatch edge 0.5)
     (priority 3)
-    (connect_pads (clearance 0.25))
-    (min_thickness 0.25) (filled_areas_thickness no)
+    (connect_pads (clearance 0.2))
+    (min_thickness 0.2) (filled_areas_thickness no)
     (fill yes (thermal_gap 0.5) (thermal_bridge_width 0.5))
     (polygon

Commit message: Update
Parts:
- added Q1: NMOS, Package_TO_SOT_SMD:SOT-23, F.Cu at (136.3, 98.9)
- added Q2: NMOS, Package_TO_SOT_SMD:SOT-23, F.Cu at (126.7, 115.2)
- added Q3: NMOS, Package_TO_SOT_SMD:SOT-23, F.Cu at (148.0, 90.2)
- added Q4: NMOS, Package_TO_SOT_SMD:SOT-23, F.Cu at (119.2, 89.5)
- added Q6: NMOS, Package_TO_SOT_SMD:SOT-23, F.Cu at (138.3, 115.0)
- added Q7: NMOS, Package_TO_SOT_SMD:SOT-23, F.Cu at (132.0, 115.2)
- moved C14 0.29 mm to (132.1, 111.5)
- renumbered C18 to C10, C19 to C11, C20 to C12, C21 to C13, C22 to C14, C23 to C15, C24 to C16, C25 to C17, C14 to C8, C15 to C9, F4 to F2, F5 to F3, F2 to F4, F3 to F5, J3 to J2, J8 to J3, J7 to J4, J16 to J5, J4 to J6, J2 to J7, J15 to J8, JP3 to JP2, JP2 to JP3, D4 to PWR
Connections:
- J1 pad 3: /GPIO_SPLY_2 -> /GPIO_GND_2
- J1 pad 4: /GPIO_SPLY_2 -> /GPIO_GND_2
- J2 pad 1: /GPIO_SPLY_5 -> /GPIO_GND_5
- J2 pad 11: GND -> +5V
- J2 pad 12: GND -> +5V
- J2 pad 13: GND -> +5V
- J2 pad 14: GND -> +5V
- J2 pad 15: /GPIO_SPLY_7 -> GND
- J2 pad 16: /GPIO_SPLY_7 -> GND
- J2 pad 17: /GPIO_SPLY_8 -> GND
- J2 pad 18: /GPIO_SPLY_8 -> GND
- J2 pad 2: /GPIO_SPLY_5 -> /GPIO_GND_5
- J2 pad 3: /GPIO_SPLY_6 -> /GPIO_GND_6
- J2 pad 4: /GPIO_SPLY_6 -> /GPIO_GND_6
- J6 pad 1: GND -> +5V
- J6 pad 17: /GPIO_SPLY_3 -> /GPIO_GND_3
- J6 pad 18: /GPIO_SPLY_3 -> /GPIO_GND_3
- J6 pad 19: /GPIO_SPLY_4 -> /GPIO_GND_4
- J6 pad 2: GND -> +5V
- J6 pad 20: /GPIO_SPLY_4 -> /GPIO_GND_4
- J6 pad 3: GND -> +5V
- J6 pad 4: GND -> +5V
- J7 pad 3: /GPIO_SPLY_1 -> /GPIO_GND_1
- J7 pad 4: /GPIO_SPLY_1 -> /GPIO_GND_1
- U5 pad 33: /GPIO_SPLY_1 -> Net-(Q2-G)
- U5 pad 34: /GPIO_SPLY_2 -> Net-(Q4-G)
- U5 pad 35: /GPIO_SPLY_3 -> Net-(Q6-G)
- U5 pad 36: /GPIO_SPLY_4 -> Net-(Q7-G)
- U5 pad 37: /GPIO_SPLY_5 -> Net-(Q1-G)
- U5 pad 38: /GPIO_SPLY_6 -> Net-(Q3-G)
- U5 pad 39: /GPIO_SPLY_7 -> unconnected-(U5-PC8-Pad39)
- U5 pad 40: /GPIO_SPLY_8 -> unconnected-(U5-PC9-Pad40)
Routing:
- net /GPIO_SPLY_1: track 71.1 -> 0.00 mm, vias 2 -> 0
- net /GPIO_SPLY_4: track 65.3 -> 0.00 mm, vias 2 -> 0
- net /GPIO_SPLY_3: track 60.8 -> 0.00 mm, vias 2 -> 0
- net /GPIO_GND_1: track 0.00 -> 50.7 mm
- net /GPIO_GND_3: track 0.00 -> 50.4 mm
- net /GPIO_SPLY_5: track 49.8 -> 0.00 mm, vias 2 -> 0
- net /GPIO_GND_4: track 0.00 -> 49.2 mm
- net /GPIO_SPLY_6: track 47.9 -> 0.00 mm, vias 2 -> 0
- net /GPIO_GND_5: track 0.00 -> 39.0 mm, vias 0 -> 2
- net /GPIO_SPLY_7: track 36.9 -> 0.00 mm
- net /GPIO_SPLY_8: track 35.0 -> 0.00 mm
- net Net-(Q6-G): track 0.00 -> 27.7 mm, vias 0 -> 2
- net Net-(Q3-G): track 0.00 -> 26.0 mm, vias 0 -> 2
- net /GPIO_SPLY_2: track 24.3 -> 0.00 mm, vias 1 -> 0
- net Net-(Q7-G): track 0.00 -> 23.8 mm, vias 0 -> 2
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Other:
- outline, holes or cut-outs redrawn
- board text added: "5V"
- board text added: "5|24"
- board text added: "ADC1"
- board text added: "ADC2"
- board text added: "ADC3"
- board text added: "ADC4"
- board text added: "ADC5"
- board text added: "ADC6"
- board text added: "ADC7"
- board text added: "ADC8"
- board text added: "BATIN"
- board text added: "CANH"
- board text added: "CANL"
- board text added: "DSUP"
- board text added: "GND"
- board text added: "GPIO1"
- board text added: "GPIO2"
- board text added: "GPIO3"
- board text added: "GPIO4"
- board text added: "GPIO5"
- board text added: "GPIO6"
- board text added: "MISO"
- board text added: "MOSI"
- board text added: "SCL"
- board text added: "SCLK"
- board text added: "SDA"
- board text added: "SUP1"
- board text added: "SUP2"
- board text added: "SUP3"
- board text added: "SUP4"
- board text added: "SUP5"
- board text added: "SUP6"
- board text added: "SUP7"
- board text added: "SUP8"
- board text added: "U_RX"
- board text added: "U_TX"
- board text added: "~{CS}"
