File: VMU/POWER.kicad_sch (KiCad schematic)
At the start: 28 parts

Commit message: sdfsd
Parts:
- removed C? (x6): 10n, Capacitor_SMD:C_0603_1608Metric_Pad1.08x0.95mm_HandSolder, symbol Device:C
- JP1: footprint Connector_PinHeader_2.54mm:PinHeader_1x03_P2.54mm_Vertical -> Jumper:SolderJumper-3_P2.0mm_Open_TrianglePad1.0x1.5mm_NumberLabels

Commit message: Adad
a
Other:
- moved on the sheet: C?, D?, F4, F?, FB1, R?, U?, VR?

Commit message: RoutingV2
Connections:
- net SUPPLY_5 renamed PB_SUPPLY
Changed lines of the file:
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@@
   (junction (at 165.735 46.99) (diameter 0) (color 0 0 0 0)
   )
+  (junction (at 199.39 130.81) (diameter 0) (color 0 0 0 0)
+  )
   (junction (at 226.06 124.46) (diameter 0) (color 0 0 0 0)
   )
-  (junction (at 226.06 127.635) (diameter 0) (color 0 0 0 0)
-  )
   (junction (at 137.795 143.51) (diameter 0) (color 0 0 0 0)
   )
@@
     (stroke (width 0) (type default))
   )
-  (wire (pts (xy 226.06 127.635) (xy 226.06 130.81))
-    (stroke (width 0) (type default))
-  )
   (wire (pts (xy 196.215 126.365) (xy 199.39 126.365))
     (stroke (width 0) (type default))
@@
     (stroke (width 0) (type default))
   )
+  (wire (pts (xy 199.39 133.985) (xy 206.375 133.985))
+    (stroke (width 0) (type default))
+  )
   (wire (pts (xy 236.22 50.165) (xy 236.22 52.705))
     (stroke (width 0) (type default))
@@
     (stroke (width 0) (type default))
   )
+  (wire (pts (xy 199.39 130.81) (xy 199.39 133.985))
+    (stroke (width 0) (type default))
+  )
   (wire (pts (xy 106.68 59.69) (xy 111.76 59.69))
     (stroke (width 0) (type default))
@@
   )
   (wire (pts (xy 171.45 43.18) (xy 171.45 46.99))
-    (stroke (width 0) (type default))
-  )
-  (wire (pts (xy 226.06 130.81) (xy 231.775 130.81))
     (stroke (width 0) (type default))
   )
@@
     (effects (font (size 1.27 1.27)) (justify left))
   )
-  (hierarchical_label "PB_SUPPLY" (shape output) (at 231.775 130.81 0) (fields_autoplaced)
-    (effects (font (size 1.27 1.27)) (justify left))
-  )
+  (hierarchical_label "PB_SUPPLY" (shape output) (at 206.375 133.985 0) (fields_autoplaced)
+    (effects (font (size 1.27 1.27)) (justify left))
+  )

Commit message: Update
Parts:
- renumbered F4 to F2, F5 to F3, F2 to F4, F3 to F5

Commit message: banana
Parts:
- gave numbers to parts that had none: 13
- renumbered JP1 to JP2, JP1 to JP3, JP1 to JP4
