File: VMU/MCU.kicad_sch (KiCad schematic)
At the start: 27 parts, among them J1 ARM_JTAG_SWD_10, U1 SN65HVD233, U2 STM32F091RCTx, Y1 Crystal_GND24

Commit message: sdfsd
Connections:
- net GPIO_SPLY_1: now reaches U2.33 (PB12)
- net GPIO_SPLY_2: now reaches U2.34 (PB13)
- net GPIO_SPLY_3: now reaches U2.35 (PB14)
- net GPIO_SPLY_4: now reaches U2.36 (PB15)
- net GPIO_SPLY_5: now reaches U2.37 (PC6)
- net GPIO_SPLY_6: now reaches U2.38 (PC7)
- net GPIO_SPLY_7: now reaches U2.39 (PC8)
- net GPIO_SPLY_8: now reaches U2.40 (PC9)
- no-connect marks 30 -> 21
Changed lines of the file:
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@@
   (title_block
     (title "VEHICLE MEASUREMENT SYSTEM (VMU)")
+    (date "2020-05-05")
     (rev "1.0")
     (company "KTH FORMULA STUDENT")
-    (comment 1 "DeV18")
+    (comment 1 "Dev18")
     (comment 2 "FILIP SVEBECK")
     (comment 3 "FSVEBECK@KTH.SE")
@@
   (no_connect (at 142.24 132.715))
   (no_connect (at 175.26 107.315))
-  (no_connect (at 142.24 122.555))
   (no_connect (at 142.24 130.175))
   (no_connect (at 175.26 112.395))
   (no_connect (at 175.26 109.855))
   (no_connect (at 142.24 135.255))
-  (no_connect (at 175.26 135.255))
   (no_connect (at 54.61 88.265))
   (no_connect (at 175.26 79.375))
@@
   (no_connect (at 142.24 92.075))
   (no_connect (at 142.24 137.795))
-  (no_connect (at 142.24 125.095))
-  (no_connect (at 175.26 132.715))
   (no_connect (at 54.61 90.805))
   (no_connect (at 175.26 125.095))
   (no_connect (at 142.24 140.335))
-  (no_connect (at 142.24 117.475))
   (no_connect (at 175.26 97.155))
   (no_connect (at 175.26 114.935))
-  (no_connect (at 175.26 137.795))
-  (no_connect (at 142.24 112.395))
-  (no_connect (at 142.24 120.015))
-  (no_connect (at 175.26 140.335))
   (wire (pts (xy 21.59 170.18) (xy 21.59 166.37))
     (stroke (width 0) (type default))
@@
     (stroke (width 0) (type default))
   )
+  (wire (pts (xy 196.85 132.715) (xy 175.26 132.715))
+    (stroke (width 0) (type default))
+  )
   (wire (pts (xy 45.72 123.825) (xy 40.64 123.825))
     (stroke (width 0) (type default))
@@
   )
   (wire (pts (xy 47.625 23.495) (xy 45.085 23.495))
+    (stroke (width 0) (type default))
+  )
+  (wire (pts (xy 142.24 122.555) (xy 120.65 122.555))
     (stroke (width 0) (type default))
   )
@@
     (stroke (width 0) (type default))
   )
+  (wire (pts (xy 142.24 120.015) (xy 120.65 120.015))
+    (stroke (width 0) (type default))
+  )
   (wire (pts (xy 187.96 81.915) (xy 175.26 81.915))
     (stroke (width 0) (type default))
@@
   )
   (wire (pts (xy 67.31 181.61) (xy 77.47 181.61))
+    (stroke (width 0) (type default))
+  )
+  (wire (pts (xy 142.24 117.475) (xy 120.65 117.475))
     (stroke (width 0) (type default))
   )
@@
     (stroke (width 0) (type default))
   )
+  (wire (pts (xy 175.26 140.335) (xy 196.85 140.335))
+    (stroke (width 0) (type default))
+  )
   (wire (pts (xy 175.26 102.235) (xy 200.025 102.235))
     (stroke (width 0) (type default))
@@
     (stroke (width 0) (type default))
   )
+  (wire (pts (xy 120.65 125.095) (xy 142.24 125.095))
+    (stroke (width 0) (type default))
+  )
   (wire (pts (xy 175.26 84.455) (xy 187.96 84.455))
     (stroke (width 0) (type default))
@@
     (stroke (width 0) (type default))
   )
+  (wire (pts (xy 175.26 137.795) (xy 196.85 137.795))
+    (stroke (width 0) (type default))
+  )
   (wire (pts (xy 77.47 166.37) (xy 87.63 166.37))
     (stroke (width 0) (type default))
@@
   )
   (wire (pts (xy 34.925 34.925) (xy 24.765 34.925))
+    (stroke (width 0) (type default))
+  )
+  (wire (pts (xy 175.26 135.255) (xy 196.85 135.255))
     (stroke (width 0) (type default))
   )
@@
     (effects (font (size 1.27 1.27)) (justify left))
   )
+  (hierarchical_label "GPIO_SPLY_2" (shape input) (at 196.85 135.255 0) (fields_autoplaced)
+    (effects (font (size 1.27 1.27)) (justify left))
+  )
+  (hierarchical_label "GPIO_SPLY_4" (shape input) (at 196.85 140.335 0) (fields_autoplaced)
+    (effects (font (size 1.27 1.27)) (justify left))
+  )
+  (hierarchical_label "GPIO_SPLY_1" (shape input) (at 196.85 132.715 0) (fields_autoplaced)
+    (effects (font (size 1.27 1.27)) (justify left))
+  )
+  (hierarchical_label "GPIO_SPLY_5" (shape input) (at 120.65 117.475 180) (fields_autoplaced)
+    (effects (font (size 1.27 1.27)) (justify right))
+  )
   (hierarchical_label "ANALOG_6" (shape input) (at 187.96 61.595 0) (fields_autoplaced)
     (effects (font (size 1.27 1.27)) (justify left))
@@
     (effects (font (size 1.27 1.27)) (justify left))
   )
+  (hierarchical_label "GPIO_SPLY_7" (shape input) (at 120.65 122.555 180) (fields_autoplaced)
+    (effects (font (size 1.27 1.27)) (justify right))
+  )
   (hierarchical_label "CAN1_L" (shape bidirectional) (at 75.565 40.64 0) (fields_autoplaced)
     (effects (font (size 1.27 1.27)) (justify left))
@@
   (hierarchical_label "ANALOG_7" (shape input) (at 187.96 64.135 0) (fields_autoplaced)
     (effects (font (size 1.27 1.27)) (justify left))
+  )
+  (hierarchical_label "GPIO_SPLY_8" (shape input) (at 120.65 125.095 180) (fields_autoplaced)
+    (effects (font (size 1.27 1.27)) (justify right))
   )
   (hierarchical_label "ANALOG_8" (shape input) (at 187.96 66.675 0) (fields_autoplaced)
@@
     (effects (font (size 1.27 1.27)) (justify right))
   )
+  (hierarchical_label "GPIO_SPLY_3" (shape input) (at 196.85 137.795 0) (fields_autoplaced)
+    (effects (font (size 1.27 1.27)) (justify left))
+  )
   (hierarchical_label "I2C_SCL" (shape input) (at 197.485 117.475 0) (fields_autoplaced)
     (effects (font (size 1.27 1.27)) (justify left))
@@
     (effects (font (size 1.27 1.27)) (justify left))
   )
+  (hierarchical_label "GPIO_SPLY_6" (shape input) (at 120.65 120.015 180) (fields_autoplaced)
+    (effects (font (size 1.27 1.27)) (justify right))
+  )
   (hierarchical_label "SPI_SCLK" (shape input) (at 187.96 71.755 0) (fields_autoplaced)

Commit message: RoutingV2
Parts:
- removed C11, C14: 36pF, Capacitor_SMD:C_0603_1608Metric_Pad1.08x0.95mm_HandSolder, symbol Device:C
- removed R6: 0, Resistor_SMD:R_0603_1608Metric_Pad0.98x0.95mm_HandSolder, symbol Device:R
- removed Y1: Crystal_GND24, Crystal:Crystal_SMD_3225-4Pin_3.2x2.5mm_HandSoldering, symbol Device:Crystal_GND24
Connections:
- net ANALOG_1: now also U2.17 (PA3); no longer U2.8 (PC0)
- net ANALOG_2: now also U2.16 (PA2); no longer U2.9 (PC1)
- net ANALOG_3: now also U2.15 (PA1); no longer U2.10 (PC2)
- net ANALOG_4: now also U2.14 (PA0); no longer U2.11 (PC3)
- net ANALOG_5: now also U2.11 (PC3); no longer U2.14 (PA0)
- net ANALOG_6: now also U2.10 (PC2); no longer U2.15 (PA1)
- net ANALOG_7: now also U2.9 (PC1); no longer U2.16 (PA2)
- net ANALOG_8: now also U2.8 (PC0); no longer U2.17 (PA3)
Other:
- note removed: "25 MHz EXTERNAL OSCILLATOR"

Commit message: fiixes
Parts:
- added Q1: NMOS, symbol Simulation_SPICE:NMOS
Connections:
- net GND: now also Q1.3 (S)
- net GPIO_SPLY_4: no longer names the net of U2.36 (PB15)
- net GPIO_SPLY_4: now also Q1.2 (G)
- new net GPIO_GND_4: Q1.1 (D)
Changed lines of the file:
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@@
+    (stroke (width 0) (type default))
+  )
+  (wire (pts (xy 175.26 140.335) (xy 219.075 140.335))
     (stroke (width 0) (type default))
   )
@@
     (stroke (width 0) (type default))
   )
+  (wire (pts (xy 227.33 132.715) (xy 226.695 132.715))
+    (stroke (width 0) (type default))
+  )
   (wire (pts (xy 142.24 109.855) (xy 128.905 109.855))
     (stroke (width 0) (type default))
@@
     (stroke (width 0) (type default))
   )
+  (wire (pts (xy 226.695 145.415) (xy 226.695 147.32))
+    (stroke (width 0) (type default))
+  )
   (wire (pts (xy 67.31 181.61) (xy 77.47 181.61))
     (stroke (width 0) (type default))
@@
   )
   (wire (pts (xy 45.085 23.495) (xy 45.085 19.685))
+    (stroke (width 0) (type default))
+  )
+  (wire (pts (xy 226.695 132.715) (xy 226.695 135.255))
     (stroke (width 0) (type default))
   )
   (polyline (pts (xy 13.589 60.579) (xy 91.567 60.579))
     (stroke (width 0) (type dash))
-  )
-  (wire (pts (xy 175.26 140.335) (xy 196.85 140.335))
-    (stroke (width 0) (type default))
   )
   (wire (pts (xy 175.26 102.235) (xy 200.025 102.235))
@@
     (effects (font (size 1.27 1.27)) (justify left))
   )
-  (hierarchical_label "GPIO_SPLY_4" (shape input) (at 196.85 140.335 0) (fields_autoplaced)
+  (hierarchical_label "GPIO_GND_4" (shape input) (at 227.33 132.715 0) (fields_autoplaced)
     (effects (font (size 1.27 1.27)) (justify left))
   )
@@
     )
   )
+  (symbol (lib_id "power:GND") (at 226.695 147.32 0) (unit 1)
+    (in_bom yes) (on_board yes) (dnp no) (fields_autoplaced)
+    (property "Reference" "#PWR034" (at 226.695 153.67 0)
+      (effects (font (size 1.27 1.27)) hide)
+    )
+    (property "Value" "GND" (at 226.695 151.765 0)
+      (effects (font (size 1.27 1.27)))
+    )
+    (property "Footprint" "" (at 226.695 147.32 0)
+      (effects (font (size 1.27 1.27)) hide)
+    )
+    (property "Datasheet" "" (at 226.695 147.32 0)
+      (effects (font (size 1.27 1.27)) hide)
+    )
+    (pin "1")
+    (instances
+      (project "VMU"
+        (path "/a0b206d8-cab6-473c-9bbb-e8da011ef93c/00000000-0000-0000-0000-00005eb3d0bc"
+          (reference "#PWR034") (unit 1)
+        )
+      )
+    )
+  )
   (symbol (lib_id "power:+3.3V") (at 160.02 47.625 0) (unit 1)
     (in_bom yes) (on_board yes) (dnp no) (fields_autoplaced)
@@
         )
       )
+    )
+  )
+  (symbol (lib_id "Simulation_SPICE:NMOS") (at 224.155 140.335 0) (unit 1)
+    (in_bom yes) (on_board yes) (dnp no) (fields_autoplaced)
+    (property "Reference" "Q1" (at 229.87 139.065 0)
+      (effects (font (size 1.27 1.27)) (justify left))
+    )
+    (property "Value" "NMOS" (at 229.87 141.605 0)
+      (effects (font (size 1.27 1.27)) (justify left))
+    )
+    (property "Footprint" "" (at 229.235 137.795 0)
+      (effects (font (size 1.27 1.27)) hide)
+    )
+    (property "Datasheet" "https://ngspice.sourceforge.io/docs/ngspice-manual.pdf" (at 224.155 153.035 0)
+      (effects (font (size 1.27 1.27)) hide)
+    )
+    (property "Sim.Device" "NMOS" (at 224.155 157.48 0)
+      (effects (font (size 1.27 1.27)) hide)
+    )
+    (property "Sim.Type" "VDMOS" (at 224.155 159.385 0)
+      (effects (font (size 1.27 1.27)) hide)
+    )
+    (property "Sim.Pins" "1=D 2=G 3=S" (at 224.155 155.575 0)
+      (effects (font (size 1.27 1.27)) hide)
+    )
+    (pin "1")
+    (pin "2")
+    (pin "3")
+    (instances
+      (project "VMU"
+        (path "/a0b206d8-cab6-473c-9bbb-e8da011ef93c/00000000-0000-0000-0000-00005eb3d0bc"
+          (reference "Q1") (unit 1)
+        )
+      )

Commit message: Update
Parts:
- added Q1, Q2, Q3, Q4, Q6: NMOS, Package_TO_SOT_SMD:SOT-23, symbol Simulation_SPICE:NMOS
- Q7: renamed from Q1; footprint (none) -> Package_TO_SOT_SMD:SOT-23
Connections:
- net GND: now also Q1.3 (S), Q2.3 (S), Q3.3 (S), Q4.3 (S), Q6.3 (S)
- net GPIO_SPLY_1: no longer names the net of U2.33 (PB12)
- net GPIO_SPLY_1: now also Q2.2 (G)
- net GPIO_SPLY_2: no longer names the net of U2.34 (PB13)
- net GPIO_SPLY_2: now also Q4.2 (G)
- net GPIO_SPLY_3: no longer names the net of U2.35 (PB14)
- net GPIO_SPLY_3: now also Q6.2 (G)
- net GPIO_SPLY_5: no longer names the net of U2.37 (PC6)
- net GPIO_SPLY_5: now also Q1.2 (G)
- net GPIO_SPLY_6: no longer names the net of U2.38 (PC7)
- net GPIO_SPLY_6: now also Q3.2 (G)
- net GPIO_SPLY_7: no longer names the net of U2.39 (PC8)
- net GPIO_SPLY_8: no longer names the net of U2.40 (PC9)
- new net GPIO_GND_1: Q2.1 (D)
- new net GPIO_GND_2: Q4.1 (D)
- new net GPIO_GND_3: Q6.1 (D)
- new net GPIO_GND_5: Q1.1 (D)
- new net GPIO_GND_6: Q3.1 (D)
- no-connect marks 21 -> 23
Other:
- moved on the sheet: C1, C2, C3, C5, C6, C7, C8, C9, Q7

Commit message: Merge branch 'DeV20_development'
Parts:
- renumbered C1 to C10, C2 to C11, C3 to C12, C5 to C13, C6 to C14, C7 to C15, C8 to C16, C9 to C17, C4 to C8, C10 to C9, D2 to D5, D1 to D6, D2 to D7, J1 to J8, R1 to R2, R1 to R3, R46 to R4, R45 to R5, R46 to R6, R1 to R7, R1 to R8, U1 to U4, U2 to U5
