File: VMU/VMU.kicad_sch (KiCad schematic)
At the start: 6 parts, among them J1 TBL009-254-14GY-2GY, J3 Conn_01x08_Pin, J4 Conn_01x08_Pin, J5 Conn_01x02_Pin, J7 TBL009-254-14GY-2GY, U2 TLV9064

Commit message: Merge branch 'DeV20_development'
Parts:
- added C1, C2: 100n, Capacitor_SMD:C_0603_1608Metric_Pad1.08x0.95mm_HandSolder, symbol Device:C
- added J2, J6: TBL009-254-14GY-2GY, KTHFS:TBL00925414GY2GY, symbol realTBL009-254-14GY-2GY:TBL009-254-14GY-2GY
- added U1: TLV9064, Package_SO:SOIC-14_3.9x8.7mm_P1.27mm, symbol Amplifier_Operational:TLV9064
- added unit 5 of U2
- added unit 1 of U2
- added unit 2 of U2
Connections:
- net DIGITAL_SUPPLY_1: now also J2.5, J2.6
- net DIGITAL_SUPPLY_2: now also J2.19, J2.20
- net DIGITAL_SUPPLY_3: now also J6.15, J6.16
- net GND: now also C1.2, C2.2, J2.17, J2.18, J2.27, J2.28, J6.21, J6.22, J6.5, J6.6, U1.11 (V-), U2.11 (V-)
- net battery_in: now also J6.27, J6.28
- net MCU/ANALOG_8: now reaches U2.13 (-)
- net MCU/ANALOG_8: now also U2.14
- net at J4.1 (Pin_1): now also U1.3 (+)
- net at J4.2 (Pin_2): now also U1.5 (+)
- net at J4.3 (Pin_3): now also U1.10 (+)
- net at J4.4 (Pin_4): now also U1.12 (+)
- net at J4.5 (Pin_5): now also U2.3 (+)
- net at J4.6 (Pin_6): now also U2.5 (+)
- net MCU/ANALOG_7: now reaches U2.8
- net MCU/ANALOG_7: now also U2.9 (-)
- new net +24V: J2.15, J2.16
- new net +3.3V: J2.25, J2.26
- new net +5V: C1.1, C2.1, J2.11, J2.12, J2.13, J2.14, J6.1, J6.2, J6.3, J6.4, U1.4 (V+), U2.4 (V+)
- new net CAN1_H: J6.25, J6.26
- new net CAN1_L: J6.23, J6.24
- new net GPIO_GND_3: J6.17, J6.18
- new net GPIO_GND_4: J6.19, J6.20
- new net GPIO_GND_5: J2.1, J2.2
- new net GPIO_GND_6: J2.3, J2.4
- new net I2C_SCL: J2.10, J2.9
- new net I2C_SDA: J2.7, J2.8
- new net MCU/ANALOG_1: U1.1, U1.2 (-)
- new net MCU/ANALOG_2: U1.6 (-), U1.7
- new net MCU/ANALOG_3: U1.8, U1.9 (-)
- new net MCU/ANALOG_4: U1.13 (-), U1.14
- new net MCU/ANALOG_5: U2.1, U2.2 (-)
- new net MCU/ANALOG_6: U2.6 (-), U2.7
- new net SPI_MISO: J6.13, J6.14
- new net SPI_MOSI: J6.11, J6.12
- new net SPI_SCLK: J6.10, J6.9
- new net SPI_~{CS}: J6.7, J6.8
- new net UART_RX: J2.21, J2.22
- new net UART_TX: J2.23, J2.24
Other:
- added sheet MCU (MCU.kicad_sch)
- sheet POWER ports: added SUPPLY_1; removed none
- note added: "OP AMP SUPPLYy"
- note added: "To rear distribution board right"
